File: KiCad/BallValveController.kicad_pcb (KiCad board)
At the start: 2 copper layers, 55.6 x 43.2 mm, 60 parts, among them J1 Screw_Terminal_01x03, J2 Screw_Terminal_01x04, J3 Screw_Terminal_01x04, J4 Screw_Terminal_01x04, J6 Screw_Terminal_01x04, J7 Screw_Terminal_01x02, J8 ME3116 in-gnd-out, K1 G5V-2, Q1 Q_PMOS_GDS, Q2 2N2222A, U3 XIAO-ESP32-C6, U4 TPS561201/08 or TPS563200

Commit message: DRC + design rules updates
Parts:
- moved J8 1.36 mm to (156.4, 97.5)
- moved C6 0.92 mm to (160.5, 94.3)
- moved J1 0.24 mm to (160.9, 86.7)
- moved J7 0.18 mm to (149.1, 86.7)
Routing:
- net +3V3: track 94.0 -> 95.7 mm
- net /PwrIn: track 41.1 -> 42.5 mm
- net GND: track 162.4 -> 161.6 mm, vias 17 -> 19
- net Net-(U3-GPIO1_A1_D1): track 32.5 -> 31.8 mm
Other:
- board text added: "Valve ctl rev 8.2.0 (C)2026 Hans Rune Bue <email@hansrune.net>"
- board text added: "Valve ctl rev 8.2.0 (C)2026-Hans Rune Bue <email@hansrune.net>"
- board text removed: "Valve ctl rev 8.1.0 (C)2026 Hans Rune Bue <email@hansrune.net>"
- board text removed: "Valve ctl rev 8.1.0 (C)2026-Hans Rune Bue <email@hansrune.net>"
